Commit message: gazebo, nav stack

File: raccoon_description/urdf/raccoon.urdf.xacro (robot description, xacro)
@@ -17,5 +17,5 @@
     <xacro:property name="wheel_offset_y" value="0.0775" />
     <xacro:property name="wheel_offset_z" value="0.000" />
-    <xacro:property name="chassis_mass" value="1.200" />
+    <xacro:property name="chassis_mass" value="12.000" />
     <xacro:property name="chassis_size_x" value="0.160" />
     <xacro:property name="chassis_size_y" value="0.160" />
@@ -69,13 +69,13 @@
             <publishWheelJointState>false</publishWheelJointState>
             <alwaysOn>true</alwaysOn>
-            <updateRate>100.0</updateRate>
+            <updateRate>50.0</updateRate>
             <!-- strange gazebo annotation -->
-            <leftJoint>right_joint</leftJoint>
-            <rightJoint>left_joint</rightJoint>
+            <leftJoint>left_joint</leftJoint>
+            <rightJoint>right_joint</rightJoint>
             <wheelSeparation>${2*wheel_offset_y}</wheelSeparation>
             <wheelDiameter>${2*wheel_radius}</wheelDiameter>
             <broadcastTF>1</broadcastTF>
-            <wheelTorque>1</wheelTorque>
-            <wheelAcceleration>1.8</wheelAcceleration>
+            <wheelTorque>10</wheelTorque>
+            <wheelAcceleration>0.8</wheelAcceleration>
             <commandTopic>/raccoon_velocity_controller/cmd_vel</commandTopic>
             <publishOdomTF>false</publishOdomTF>

Commit message: fixed gazebo, added explore :)

File: raccoon_description/urdf/raccoon.urdf.xacro (robot description, xacro)
@@ -31,9 +31,9 @@
     <xacro:property name="wheel_radius" value="0.0325" />
     <xacro:property name="wheel_mount" value="0.0183" />
-    <xacro:property name="wheel_mass" value="0.200" />
+    <xacro:property name="wheel_mass" value="5.000" />
     <xacro:property name="wheel_offset_x" value="0.0" />
     <xacro:property name="wheel_offset_y" value="0.075" />
     <xacro:property name="wheel_offset_z" value="0.000" />
-    <xacro:property name="chassis_mass" value="1.000" />
+    <xacro:property name="chassis_mass" value="10.000" />
     <xacro:property name="chassis_size_x" value="0.160" />
     <xacro:property name="chassis_size_y" value="0.160" />
@@ -42,5 +42,11 @@
         <link name="base_footprint">
             <collision>
-                <origin xyz="-0.065 0 0.006" rpy="0 0 0" />
+                <origin xyz="0.065 0 0.005" rpy="0 0 0" />
+                <geometry>
+                    <sphere radius="0.005" />
+                </geometry>
+            </collision>
+            <collision>
+                <origin xyz="-0.065 0 0.005" rpy="0 0 0" />
                 <geometry>
                     <sphere radius="0.005" />
@@ -102,6 +108,6 @@
             <wheelDiameter>${2*wheel_radius}</wheelDiameter>
             <broadcastTF>1</broadcastTF>
-            <wheelTorque>10</wheelTorque>
-            <wheelAcceleration>0.8</wheelAcceleration>
+            <wheelTorque>1</wheelTorque>
+            <wheelAcceleration>1.8</wheelAcceleration>
             <commandTopic>/raccoon_velocity_controller/cmd_vel</commandTopic>
             <publishOdomTF>false</publishOdomTF>

File: raccoon_description/urdf/wheel65.urdf.xacro (robot description, xacro)
@@ -43,6 +43,6 @@
         </link>
         <gazebo reference="${lr}_wheel">
-            <mu1 value="1.0"/>
-            <mu2 value="1.0"/>
+            <mu1 value="10000.0"/>
+            <mu2 value="10000.0"/>
             <kp  value="10000000.0" />
             <kd  value="1.0" />

Commit message: added urdf of rev2

File: raccoon_description/urdf/raccoon.urdf.xacro (robot description, xacro)
@@ -58,5 +58,5 @@
                 <origin rpy="0.0 0.0 ${-M_PI_2}" xyz="0.0 0.0 ${wheel_mount}"/>
                 <geometry>
-                    <mesh filename="${path_meshes}/raccoon_body.dae"/>
+                    <mesh filename="${path_meshes}/raccoon_rev2.dae"/>
                 </geometry>
             </visual>
